File: Design1.brd (EAGLE design)
At the start: 148.5 x 150.3 mm, 17 parts

Commit message: added tracks
Routing:
- net GND: track 1282.1 -> 1479.6 mm
- net 24V_OUT: track 507.3 -> 578.5 mm
- net 12V_OUT: track 547.6 -> 613.7 mm
- net F2: track 78.1 -> 90.3 mm
Other:
- outline, holes or cut-outs redrawn
